File: Spiderfish PDB/Power-Distribution-Board/Power-Distribution-Board.kicad_pcb (KiCad board)
At the start: 2 copper layers, 95 parts, among them J1 Conn_01x04_Pin, J2 USB_B_Micro, U1 STM32L052K6T6, U10 AOZ2264NQI-11, U2 LM2596DSADJG, U3 LM2596DSADJG, U4 USBLC6-2SC6, U5 AOZ2264NQI-11, U6 AOZ2264NQI-11, U7 AOZ2264NQI-11, U8 AOZ2264NQI-11, U9 AOZ2264NQI-11

Commit message: added base design constraints and grouped pcb components
Parts:
- added C35: 4u7, Capacitor_SMD:C_0805_2012Metric_Pad1.18x1.45mm_HandSolder, F.Cu at (154.8, 241.0)
- added C36: 4u7, Capacitor_SMD:C_0805_2012Metric_Pad1.18x1.45mm_HandSolder, F.Cu at (276.7, 237.2)
- added C37: 4u7, Capacitor_SMD:C_0805_2012Metric_Pad1.18x1.45mm_HandSolder, F.Cu at (269.5, 286.0)
- added C38: 4u7, Capacitor_SMD:C_0805_2012Metric_Pad1.18x1.45mm_HandSolder, F.Cu at (175.0, 292.0)
- added C39: 4u7, Capacitor_SMD:C_0805_2012Metric_Pad1.18x1.45mm_HandSolder, F.Cu at (170.0, 352.8)
- added C40: 4u7, Capacitor_SMD:C_0805_2012Metric_Pad1.18x1.45mm_HandSolder, F.Cu at (245.3, 354.8)
- added J3: TB002-500-02BE, Power_Distribution_Board:TB002-500-02BE, F.Cu at (152.0, 235.2)
- added J4: TB002-500-02BE, Power_Distribution_Board:TB002-500-02BE, F.Cu at (244.8, 225.5)
- added J5: TB002-500-02BE, Power_Distribution_Board:TB002-500-02BE, F.Cu at (155.5, 294.8)
- added J6: TB002-500-02BE, Power_Distribution_Board:TB002-500-02BE, F.Cu at (235.0, 280.5)
- added J7: TB002-500-02BE, Power_Distribution_Board:TB002-500-02BE, F.Cu at (148.0, 354.8)
- added J8: TB002-500-02BE, Power_Distribution_Board:TB002-500-02BE, F.Cu at (217.8, 349.1)
- added J9: XT90PW-F, Power_Distribution_Board:XT90PWF, F.Cu at (96.2, -51.2)
- J2: footprint Connector_USB:USB_Micro-B_Wuerth_629105150521 -> Power_Distribution_Board:629105150521
- moved R31 401.4 mm to (231.4, 365.2)
- moved R34 392.6 mm to (226.7, 365.3)
- moved R36 392.4 mm to (226.7, 370.0)
- moved R37 392.3 mm to (231.4, 370.0)
- moved R29 391.8 mm to (226.4, 374.8)
- moved U10 384.1 mm to (221.3, 359.8)
- moved R32 376.9 mm to (153.0, 373.2)
- moved R33 375.9 mm to (157.7, 373.2)
- moved R35 374.4 mm to (152.7, 378.2)
- moved R28 370.3 mm to (157.8, 378.5)
- moved R30 368.2 mm to (152.4, 383.0)
- moved C25 365.9 mm to (232.4, 350.5)
- moved U9 364.5 mm to (150.6, 364.2)
- moved C27 364.4 mm to (238.0, 350.5)
- moved C31 363.7 mm to (237.8, 356.5)
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Connections:
- net /LX12V_1 renamed /12V_LX_1
- net /LX12V_2 renamed /12V_LX_2
- net /LX5V_1 renamed /5V_LX_1
- net /LX5V_2 renamed /5V_LX_2
- net /LX9V_1 renamed /9V_LX_1
- net /LX9V_2 renamed /9V_LX_2
- net Net-(C12-Pad1) renamed /12V_OUT_2
- net Net-(C13-Pad1) renamed /12V_OUT1
- net Net-(C20-Pad1) renamed /9V_OUT_1
- net Net-(C22-Pad1) renamed /9V_OUT_2
- net Net-(C28-Pad1) renamed /5V_OUT_1
- net Net-(C30-Pad1) renamed /5V_OUT_2
- net Net-(D1-K) renamed /5V_L
- net Net-(D2-K) renamed /3V3_L
- net Net-(J2-VBUS) renamed /USB_VBUS
- net Net-(U1-PA0) renamed /5V_EN_1
- net Net-(U1-PA1) renamed /9V_EN_1
- net Net-(U1-PA2) renamed /12V_EN_1
- net Net-(U1-PA3) renamed /5V_EN_2
- net Net-(U1-PA4) renamed /9V_EN_2
- net Net-(U1-PA5) renamed /12V_EN_2
- net Net-(U1-PA9) renamed /USB_ACK
- net Net-(U10-BST) renamed /5V_BST_2
- net Net-(U10-FB) renamed /5V_FB_2
- net Net-(U10-OCS) renamed /5V_OSC_2
- net Net-(U10-SS) renamed /5V_SS_2
- net Net-(U10-TON) renamed /5V_TON_2
- net Net-(U5-BST) renamed /12V_BST_2
- net Net-(U5-FB) renamed /12V_FB_2
- net Net-(U5-OCS) renamed /12V_OSC_2
- net Net-(U5-SS) renamed /12V_SS_2
- net Net-(U5-TON) renamed /12V_TON_2
- net Net-(U6-BST) renamed /12V_BST_1
- net Net-(U6-FB) renamed /12V_FB_1
- net Net-(U6-OCS) renamed /12V_OSC_1
- net Net-(U6-SS) renamed /12V_SS_1
- net Net-(U6-TON) renamed /12V_TON_1
- net Net-(U7-BST) renamed /9V_BST_1
- net Net-(U7-FB) renamed /9V_FB_1
- net Net-(U7-OCS) renamed /9V_OSC_1
- net Net-(U7-SS) renamed /9V_SS_1
- net Net-(U7-TON) renamed /9V_TON_1
- net Net-(U8-BST) renamed /9V_BST_2
- net Net-(U8-FB) renamed /9V_FB_2
- net Net-(U8-OCS) renamed /9V_OSC_2
- net Net-(U8-SS) renamed /9V_SS_2
- net Net-(U8-TON) renamed /9V_TON_2
- net Net-(U9-BST) renamed /5V_BST_1
- net Net-(U9-FB) renamed /5V_FB_1
- net Net-(U9-OCS) renamed /5V_OSC_1
- net Net-(U9-SS) renamed /5V_SS_1
- net Net-(U9-TON) renamed /5V_TON_1
- C16 pad 1: +5V -> +14V8
- C17 pad 1: +5V -> +14V8
- C2 pad 1: +5V -> /5V_FB
- C24 pad 1: +5V -> +14V8
- C25 pad 1: +5V -> +14V8
- C5 pad 1: +3V3 -> /3V3_FB
- C8 pad 1: +5V -> +14V8
- C9 pad 1: +5V -> +14V8
- J2 pad 2: Net-(J2-D-) -> /USB_USB_D-
- J2 pad 3: Net-(J2-D+) -> /USB_USB_D+
- R1 pad 1: +5V -> /5V_FB
- R10 pad 1: +3V3 -> +14V8
- R11 pad 1: +3V3 -> +14V8
- R18 pad 2: Net-(U7-PGOOD) -> /9V_PGOOD_1
- R19 pad 2: Net-(U8-PGOOD) -> /9V_PGOOD_2
- R2 pad 2: +5V -> /5V_FB
- R20 pad 1: +3V3 -> +14V8
- R21 pad 1: +3V3 -> +14V8
- R28 pad 2: Net-(U9-PGOOD) -> /5V_PGOOD_1
- R29 pad 2: Net-(U10-PGOOD) -> /5V_PGOOD_2
- R30 pad 1: +3V3 -> +14V8
- R31 pad 1: +3V3 -> +14V8
- R4 pad 1: +3V3 -> /3V3_FB
- R6 pad 2: +3V3 -> /3V3_FB
- R8 pad 2: Net-(U5-PGOOD) -> /12V_PGOOD_2
- R9 pad 2: Net-(U6-PGOOD) -> /12V_PGOOD_1
- U1 pad 14: unconnected-(U1-PB0-Pad14) -> /12V_PGOOD_1
- U1 pad 15: unconnected-(U1-PB1-Pad15) -> /12V_PGOOD_2
- U1 pad 26: unconnected-(U1-PB3-Pad26) -> /9V_PGOOD_1
- U1 pad 27: unconnected-(U1-PB4-Pad27) -> /9V_PGOOD_2
- U1 pad 28: unconnected-(U1-PB5-Pad28) -> /5V_PGOOD_1
- U1 pad 29: unconnected-(U1-PB6-Pad29) -> /5V_PGOOD_2
- U10 pad 1: Net-(U10-PGOOD) -> /5V_PGOOD_2
- U10 pad 22: +3V3 -> +14V8
- U10 pad 24: +3V3 -> +14V8
- U10 pad 7: +3V3 -> +14V8
- U10 pad 8: +3V3 -> +14V8
- U10 pad 9: +3V3 -> +14V8
- U2 pad 4: +5V -> /5V_FB
- U3 pad 4: +3V3 -> /3V3_FB
- U4 pad 1: /USB_D- -> /USB_D+
- U4 pad 3: /USB_D+ -> /USB_D-
- U4 pad 4: Net-(J2-D+) -> /USB_USB_D-
- U4 pad 6: Net-(J2-D-) -> /USB_USB_D+
- U5 pad 1: Net-(U5-PGOOD) -> /12V_PGOOD_2
- U5 pad 22: +3V3 -> +14V8
- U5 pad 24: +3V3 -> +14V8
- U5 pad 7: +3V3 -> +14V8
- U5 pad 8: +3V3 -> +14V8
- U5 pad 9: +3V3 -> +14V8
- U6 pad 1: Net-(U6-PGOOD) -> /12V_PGOOD_1
- U6 pad 22: +3V3 -> +14V8
- U6 pad 24: +3V3 -> +14V8
- U6 pad 7: +3V3 -> +14V8
- U6 pad 8: +3V3 -> +14V8
- U6 pad 9: +3V3 -> +14V8
- U7 pad 1: Net-(U7-PGOOD) -> /9V_PGOOD_1
- U7 pad 22: +3V3 -> +14V8
- U7 pad 24: +3V3 -> +14V8
- U7 pad 7: +3V3 -> +14V8
- U7 pad 8: +3V3 -> +14V8
- U7 pad 9: +3V3 -> +14V8
- U8 pad 1: Net-(U8-PGOOD) -> /9V_PGOOD_2
- U8 pad 22: +3V3 -> +14V8
- U8 pad 24: +3V3 -> +14V8
- U8 pad 7: +3V3 -> +14V8
- U8 pad 8: +3V3 -> +14V8
- U8 pad 9: +3V3 -> +14V8
- U9 pad 1: Net-(U9-PGOOD) -> /5V_PGOOD_1
- U9 pad 22: +3V3 -> +14V8
- U9 pad 24: +3V3 -> +14V8
- U9 pad 7: +3V3 -> +14V8
- U9 pad 8: +3V3 -> +14V8
- U9 pad 9: +3V3 -> +14V8
Other:
- copper layers 2 -> 4
- rule pad_to_mask_clearance: 0 -> 0.1

Commit message: rough layout for 12V reg and mcu
Parts:
- C14, C15, R14, R15, R8, R9: moved to B.Cu
- moved R15 310.9 mm to (202.1, -36.2)
- moved R9 304.1 mm to (197.9, -36.5), turned to 180 degrees
- moved R17 296.6 mm to (198.0, -23.8)
- moved R11 293.8 mm to (195.5, -30.4), turned to 90 degrees
- moved R13 291.0 mm to (197.9, -21.8), turned to 180 degrees
- moved C15 289.9 mm to (195.5, -33.3), turned to -90 degrees
- moved R8 289.3 mm to (224.7, -35.0), turned to 180 degrees
- moved R14 284.0 mm to (230.1, -35.2)
- moved C11 282.9 mm to (203.0, -36.2), turned to 180 degrees
- moved U6 281.6 mm to (199.9, -31.9)
- moved C35 280.8 mm to (197.7, -36.5), turned to 180 degrees
- moved L4 280.5 mm to (210.3, -27.0)
- moved C13 280.3 mm to (202.5, -22.7), turned to 90 degrees
- moved C9 280.0 mm to (198.0, -27.5), turned to 180 degrees
- moved R10 278.6 mm to (223.2, -28.8), turned to 90 degrees
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
Commit message: rough layout
Parts:
- C14, C15: moved to F.Cu
- R10, R11, R18, R19, R20, R21, R23, R26, R28, R29, R30, R31, R33, R36: moved to B.Cu
- moved C6 448.0 mm to (152.5, -82.9), turned to 90 degrees
- moved L2 440.0 mm to (147.3, -74.2)
- moved U3 435.5 mm to (140.2, -89.3)
- moved R6 434.5 mm to (153.1, -90.9), turned to 180 degrees
- moved R4 428.0 mm to (149.0, -90.9), turned to 180 degrees
- moved C5 426.0 mm to (153.2, -92.9)
- moved D2 412.5 mm to (134.7, -76.4), turned to 180 degrees
- moved R29 412.2 mm to (27.0, 14.0), turned to -90 degrees
- moved R36 411.7 mm to (27.2, 9.84), turned to 90 degrees
- moved R37 405.7 mm to (39.3, 12.7), turned to 180 degrees
- moved L8 405.4 mm to (32.8, -0.07)
- moved C40 404.5 mm to (27.0, 14.2), turned to -90 degrees
- moved C4 402.8 mm to (131.5, -86.8), turned to 90 degrees
- moved R31 401.9 mm to (33.2, 15.7), turned to 180 degrees
- moved C27 401.0 mm to (27.0, 9.49), turned to 90 degrees
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