File: Spiderfish PDB/Power-Distribution-Board/Power-Distribution-Board.kicad_sch (KiCad schematic)
At the start: 108 parts, among them J1 Conn_01x04_Pin, J2 USB_B_Micro, J3 TB002-500-02BE, J4 TB002-500-02BE, J5 TB002-500-02BE, J6 TB002-500-02BE, J7 TB002-500-02BE, J8 TB002-500-02BE, J9 XT90PW-F, U1 STM32L052K6T6, U10 AOZ2264NQI-11, U2 LM2596DSADJG, U3 LM2596DSADJG, U4 USBLC6-2SC6, U5 AOZ2264NQI-11, U6 AOZ2264NQI-11, U7 AOZ2264NQI-11, U8 AOZ2264NQI-11, U9 AOZ2264NQI-11

Commit message: changed mcu and ic regulator model and refined output regulator layout
Parts:
- removed C1, C4: 100u, Capacitor_SMD:C_1210_3225Metric_Pad1.33x2.70mm_HandSolder, symbol Device:C
- removed C2, C5: 10n, Capacitor_SMD:C_0805_2012Metric_Pad1.18x1.45mm_HandSolder, symbol Device:C
- removed C3, C6: 470u, Capacitor_THT:CP_Radial_D8.0mm_P3.50mm, symbol Device:C
- removed D1, D2: SK32, Diode_SMD:D_SMC, symbol Device:D
- removed J9: XT90PW-F, Power_Distribution_Board:XT90PWF, symbol Power_Distribution_Board:XT90PW-F
- removed L1, L2: 33u, Power_Distribution_Board:SRP1038A-470M, symbol Power_Distribution_Board:SRP1038A-470M
- removed R1, R4: 10k, Resistor_SMD:R_0603_1608Metric_Pad0.98x0.95mm_HandSolder, symbol Device:R
- removed R2: 30k, Resistor_SMD:R_0603_1608Metric_Pad0.98x0.95mm_HandSolder, symbol Device:R
- removed R6: 17k2, Resistor_SMD:R_0603_1608Metric_Pad0.98x0.95mm_HandSolder, symbol Device:R
- removed U2, U3: LM2596DSADJG, Power_Distribution_Board:LM2596DSADJG, symbol Power_Distribution_Board:LM2596DSADJG
- added C41, C43, C44, C46, C47, C48: 22u, Capacitor_SMD:C_0805_2012Metric_Pad1.18x1.45mm_HandSolder, symbol Device:C
- added C42, C45: 100n, Capacitor_SMD:C_1206_3216Metric_Pad1.33x1.80mm_HandSolder, symbol Device:C
- added H1, H2, H3, H4: MountingHole, MountingHole:MountingHole_3.2mm_M3_DIN965, symbol Mechanical:MountingHole
- added J10: XT90PB-F, Power_Distribution_Board:XT90PBF, symbol Power_Distribution_Board:XT90PB-F
- added L1: 3u3, Power_Distribution_Board:IHLP-4040DZ-01, symbol Power_Distribution_Board:IHLP4040DZER3R3M01
- added L9: 4u7, Power_Distribution_Board:IHLP-4040DZ-01, symbol Power_Distribution_Board:IHLP4040DZER4R7M01
- added R38, R42: 100k, Resistor_SMD:R_0603_1608Metric_Pad0.98x0.95mm_HandSolder, symbol Device:R
- added R39: 147k, Resistor_SMD:R_0603_1608Metric_Pad0.98x0.95mm_HandSolder, symbol Device:R
- added R40, R43: 5k, Resistor_SMD:R_0603_1608Metric_Pad0.98x0.95mm_HandSolder, symbol Device:R
- added R41, R45: 20k, Resistor_SMD:R_0603_1608Metric_Pad0.98x0.95mm_HandSolder, symbol Device:R
- added R44: 91k, Resistor_SMD:R_0603_1608Metric_Pad0.98x0.95mm_HandSolder, symbol Device:R
- added U11, U12: RT6254BHGJ6F, Power_Distribution_Board:RT6254BHGJ6F, symbol Power_Distribution_Board:RT6254BHGJ6F
Connections:
- net +14V8: now also C41.1, C46.1, J10.1, R38.1, R42.1, U11.4 (VIN), U12.4 (VIN)
- net +3V3: now also C47.1, C48.1, L1.2, R44.2
- net +5V: now also C43.1, C44.1, L9.2, R39.2
- net 12V_OUT1: now also J3.2; no longer J3.1
- net 12V_OUT_2: now also J4.2; no longer J4.1
- net 9V_OUT_1: now also J5.2; no longer J5.1
- net GND: now also C12.2, C13.2, C20.2, C22.2, C28.2, C30.2, J3.1, J4.1, J5.1, J6.2, J7.2, J8.2, U10.12 (PGND_1), U10.13 (PGND_2), U10.14 (PGND_3), U10.15 (PGND_4), U5.12 (PGND_1), U5.13 (PGND_2), U5.14 (PGND_3), U5.15 (PGND_4), U6.12 (PGND_1), U6.13 (PGND_2), U6.14 (PGND_3), U6.15 (PGND_4), U7.12 (PGND_1), U7.13 (PGND_2), U7.14 (PGND_3), U7.15 (PGND_4), U8.12 (PGND_1), U8.13 (PGND_2), U8.14 (PGND_3), U8.15 (PGND_4), U9.12 (PGND_1), U9.13 (PGND_2), U9.14 (PGND_3), U9.15 (PGND_4), C41.2, C43.2, C44.2, C46.2, C47.2, C48.2, J10.2, R41.2, R45.2, U11.3 (GND), U12.3 (GND)
- removed net GNDPWR: C12.2, C13.2, C20.2, C22.2, C28.2, C30.2, J3.2, J4.2, J5.2, J6.2, J7.2, J8.2, U10.12 (PGND_1), U10.13 (PGND_2), U10.14 (PGND_3), U10.15 (PGND_4), U5.12 (PGND_1), U5.13 (PGND_2), U5.14 (PGND_3), U5.15 (PGND_4), U6.12 (PGND_1), U6.13 (PGND_2), U6.14 (PGND_3), U6.15 (PGND_4), U7.12 (PGND_1), U7.13 (PGND_2), U7.14 (PGND_3), U7.15 (PGND_4), U8.12 (PGND_1), U8.13 (PGND_2), U8.14 (PGND_3), U8.15 (PGND_4), U9.12 (PGND_1), U9.13 (PGND_2), U9.14 (PGND_3), U9.15 (PGND_4)
- new net: C42.2, L9.1, U11.5 (LX)
- new net: R38.2, U11.2 (EN)
- new net: R40.1, U11.1 (FB)
- new net: R39.1, R40.2, R41.1
- new net: R43.1, U12.1 (FB)
- new net: R42.2, U12.2 (EN)
- new net: C45.2, L1.1, U12.5 (LX)
- new net: C45.1, U12.6 (BOOT)
- new net: R43.2, R44.1, R45.1
- new net: C42.1, U11.6 (BOOT)
Other:
- moved on the sheet: J3, J4, J5
