File: Spiderfish PDB/Power-Distribution-Board/Power-Distribution-Board.kicad_sch (KiCad schematic)
At the start: 116 parts, among them J1 Conn_01x04_Pin, J10 XT90PB-F, J2 USB_B_Micro, J3 TB002-500-02BE, J4 TB002-500-02BE, J5 TB002-500-02BE, J6 TB002-500-02BE, J7 TB002-500-02BE, J8 TB002-500-02BE, U1 STM32L052K6T6, U10 AOZ2264NQI-11, U11 RT6254BHGJ6F, U12 RT6254BHGJ6F, U4 USBLC6-2SC6, U5 AOZ2264NQI-11, U6 AOZ2264NQI-11, U7 AOZ2264NQI-11, U8 AOZ2264NQI-11, U9 AOZ2264NQI-11

Commit message: rough laytout for all regs, need to increase board size to 10x10
Parts:
- removed S1: TR1-01, Power_Distribution_Board:TR101, symbol Power_Distribution_Board:TR1-01
- removed S2: EG1218, Power_Distribution_Board:EG1218, symbol Power_Distribution_Board:EG1218
- added S1: DS04-254-2-01BK-SMT, Power_Distribution_Board:DS04254201BKSMT, symbol Power_Distribution_Board:DS04-254-2-01BK-SMT
- added S2: CJS-1200TB1, Power_Distribution_Board:CJS1200TB1, symbol Power_Distribution_Board:CJS-1200TB1
- renumbered C42 to C1, C47 to C10, C48 to C11, C7 to C12, C36 to C13, C35 to C14, C10 to C15, C8 to C16, C11 to C17, C9 to C18, C12 to C19, C41 to C2, C13 to C20, C14 to C21, C15 to C22, C38 to C23, C37 to C24, C18 to C25, C16 to C26, C19 to C27, C17 to C28, C20 to C29, C43 to C3, C21 to C30, C22 to C31, C23 to C32, C39 to C33, C40 to C34, C26 to C35, C24 to C36, C27 to C37, C25 to C38, C28 to C39, C44 to C4, C29 to C40, C30 to C41, C31 to C42, C34 to C5, C33 to C6, C32 to C7, C45 to C8, C46 to C9, J10 to J2, J2 to J3, J3 to J5, J5 to J6, J6 to J7, J7 to J8, J8 to J9, L9 to L1, L1 to L2, R38 to R1, R45 to R10, R7 to R11, R8 to R12, R9 to R13, R10 to R14, R11 to R15, R12 to R16, R13 to R17, R14 to R18, R15 to R19, R40 to R2, R16 to R20, R17 to R21, R18 to R22, R19 to R23, R20 to R24, R21 to R25, R22 to R26, R23 to R27, R24 to R28, R25 to R29, R39 to R3, R26 to R30, R27 to R31, R28 to R32, R29 to R33, R30 to R34, R31 to R35, R32 to R36, R33 to R37, R34 to R38, R35 to R39, R3 to R4, R36 to R40, R37 to R41, R41 to R5, R5 to R6, R42 to R7, R43 to R8, R44 to R9, U11 to U2, U12 to U3
Connections:
- net +3V3: now also S2.1 (NO)
- net GND: now also S1.2 (NO), S2.3 (NC)
- net NRST: now also S1.1 (COM)
- net SW_BOOT0: now also S2.2 (COM)
- net 5V0_LX: now reaches C1.2, L1.1, U2.5 (LX)
- net 5V0_EN: now reaches R1.2, U2.2 (EN)
- net 5V0_FB: now reaches R2.1, U2.1 (FB)
- net 5V0_FB_R: now reaches R2.2, R3.1, R5.1
- net 3V3_FB: now reaches R8.1, U3.1 (FB)
- net 3V3_EN: now reaches R7.2, U3.2 (EN)
- net 3V3_LX: now reaches C8.2, L2.1, U3.5 (LX)
- net 3V3_BOOT: now reaches C8.1, U3.6 (BOOT)
- net 3V3_FB_R: now reaches R10.1, R8.2, R9.1
- net 5V0_BOOT: now reaches C1.1, U2.6 (BOOT)
Other:
- moved on the sheet: C2, C9, J2, R1, R2, R7, R8

Commit message: Revision A - changed 3.3V regulator to LDO - all routing done - component selection done
to do:
- update silkscreen placment
- stitching vias
Parts:
- removed C10, C11: 22u, Capacitor_SMD:C_0805_2012Metric_Pad1.18x1.45mm_HandSolder, symbol Device:C
- removed L2: 3u3, Power_Distribution_Board:IHLP-4040DZ-01, symbol Power_Distribution_Board:IHLP4040DZER3R3M01
- removed R10: 20k, Resistor_SMD:R_0603_1608Metric_Pad0.98x0.95mm_HandSolder, symbol Device:R
- removed R8: 5k, Resistor_SMD:R_0603_1608Metric_Pad0.98x0.95mm_HandSolder, symbol Device:R
- removed R9: 91k, Resistor_SMD:R_0603_1608Metric_Pad0.98x0.95mm_HandSolder, symbol Device:R
- removed U3: RT6254BHGJ6F, Power_Distribution_Board:RT6254BHGJ6F, symbol Power_Distribution_Board:RT6254BHGJ6F
- added U3: MIC5504-3.3YM5-TR, Power_Distribution_Board:MIC5504-3.3YM5-TR, symbol Power_Distribution_Board:MIC5504-3.3YM5-TR
- C5: Model GRM21BR61E106KA73K -> GRM21BZ71E106KE15L
- C8: value 100n -> 10u; footprint Capacitor_SMD:C_1206_3216Metric_Pad1.33x1.80mm_HandSolder -> Capacitor_SMD:C_0805_2012Metric_Pad1.18x1.45mm_HandSolder; Model GRM3195C2A104GA01D -> GRM21BZ71E106KE15L
- C9: value 22u -> 10u; Model CL21A226KQCLRNC -> GRM21BZ71E106KE15L
Connections:
- net 3V3_BOOT is gone; now on net +3V3: C8.1
- net 3V3_LX is gone; now on net GND: C8.2
- net +14V8: no longer C9.1, R7.1
- net +3V3: now also U3.5 (VOUT)
- net +5V: now also C9.1, R7.1, U3.1 (VIN)
- net 12V_EN_1: now also U1.10 (PA4); no longer U1.8 (PA2)
- net 12V_EN_2: now also U1.12 (PA6); no longer U1.11 (PA5)
- net 12V_PGOOD_1: now also U1.9 (PA3); no longer U1.14 (PB0)
- net 12V_PGOOD_2: now also U1.11 (PA5); no longer U1.15 (PB1)
- net 5V_EN_1: now also U1.3 (PC15_OCS32_OUT); no longer U1.6 (PA0)
- net 5V_EN_2: now also U1.28 (PB5); no longer U1.9 (PA3)
- net 5V_PGOOD_1: now also U1.2 (PC14-OCS32_IN); no longer U1.28 (PB5)
- net 5V_PGOOD_2: now also U1.27 (PB4); no longer U1.29 (PB6)
- net 9V_EN_1: now also U1.29 (PB6); no longer U1.7 (PA1)
- net 9V_EN_2: now also U1.26 (PB3); no longer U1.10 (PA4)
- net 9V_PGOOD_1: now also U1.30 (PB7); no longer U1.26 (PB3)
- net 9V_PGOOD_2: now also U1.25 (PA15); no longer U1.27 (PB4)
- net GND: now also U3.2 (GND)
- net 3V3_EN: no longer names the net of R7.2
- net 3V3_EN: now also U3.3 (EN)
Other:
- moved on the sheet: C1, C13, C14, C15, C16, C17, C18, C19, C2, C20, C21, C22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

Commit message: updated silkscreen placement + usb power switch
Parts:
- added S3: CJS-1200TB1, Power_Distribution_Board:CJS1200TB1, symbol Power_Distribution_Board:CJS-1200TB1
- R25: value 374k -> 300k; Model RT0603BRD07374KL -> ERA-3AEB304V
- R28: value 182k -> 160k; Model ERA-3AEB1823V -> RC0603FR-07160KL
- R31: value 13k -> 15k; Model ERJ-PB3B1302V -> ERA-3AEB153V
Connections:
- net +5V: now also S3.3 (NC); no longer C9.1, R7.1, U3.1 (VIN)
- net USB_VBUS: now also S3.1 (NO)
- net 9V_BST_2 renamed 7V_BST_1
- net 9V_EN_2 renamed 7V_EN_1
- net 9V_FB_2 renamed 7V_FB_1
- net 9V_LX_2 renamed 7V_LX_1
- net 9V_OSC_2 renamed 7V_OSC_1
- net 9V_OUT_2 renamed 7V_OUT_1
- net 9V_PGOOD_2 renamed 7V_PGOOD_1
- net 9V_SS_2 renamed 7V_SS_1
- net 9V_TON_2 renamed 7V_TON_1
- new net: C9.1, R7.1, S3.2 (COM), U3.1 (VIN)
Changed lines of the file:
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@@
 	)
 	(no_connect
-		(at 411.48 93.98)
+		(at 537.21 87.63)
 	)
 	(no_connect
-		(at 537.21 87.63)
+		(at 411.48 93.98)
 	)
 	(no_connect
@@
 	(wire
 		(pts
-			(xy 106.68 81.28) (xy 106.68 86.36)
-		)
-		(stroke
-			(width 0)
-			(type default)
-		)
-	)
-	(wire
-		(pts
 			(xy 462.28 82.55) (xy 469.9 82.55)
 		)
@@
 	(wire
 		(pts
+			(xy 71.12 86.36) (xy 81.28 86.36)
+		)
+		(stroke
+			(width 0)
+			(type default)
+		)
+	)
+	(wire
+		(pts
 			(xy 527.05 179.07) (xy 543.56 179.07)
 		)
@@
 	(wire
 		(pts
+			(xy 73.66 88.9) (xy 81.28 88.9)
+		)
+		(stroke
+			(width 0)
+			(type default)
+		)
+	)
+	(wire
+		(pts
 			(xy 260.35 80.01) (xy 294.64 80.01)
 		)
@@
 		)
 	)
-	(label "9V_OUT_2"
+	(label "7V_OUT_1"
 		(at 520.7 306.07 0)
 		(effects
@@
 		)
 	)
-	(label "9V_PGOOD_2"
-		(at 472.44 274.32 0)
+	(label "7V_PGOOD_1"
+		(at 472.44 275.59 0)
 		(effects
 			(font
@@
 		)
 	)
-	(label "9V_BST_2"
+	(label "7V_BST_1"
 		(at 469.9 284.48 0)
 		(effects
@@
 		)
 	)
-	(label "9V_SS_2"
+	(label "7V_SS_1"
 		(at 417.83 314.96 0)
 		(effects
@@
 		)
 	)
-	(label "9V_EN_2"
+	(label "7V_EN_1"
 		(at 416.56 304.8 0)
 		(effects
@@
 		)
 	)
-	(label "9V_LX_2"
+	(label "7V_LX_1"
 		(at 490.22 298.45 0)
 		(effects
@@
 	)
 	(label "USB_VBUS"
+		(at 71.12 86.36 0)
+		(effects
+			(font
+				(size 1.27 1.27)
+			)
+			(justify left bottom)
+		)
+	)
+	(label "USB_VBUS"
 		(at 516.89 72.39 0)
 		(effects
@@
 		)
 	)
-	(label "9V_EN_2"
+	(label "7V_EN_1"
 		(at 411.48 96.52 180)
 		(effects
@@
 		)
 	)
-	(label "9V_PGOOD_2"
+	(label "7V_PGOOD_1"
 		(at 411.48 82.55 180)
 		(effects
@@
 		)
 	)
-	(label "9V_TON_2"
+	(label "7V_TON_1"
 		(at 416.56 298.45 0)
 		(effects
@@
 		)
 	)
-	(label "9V_FB_2"
+	(label "7V_FB_1"
 		(at 485.14 316.23 0)
 		(effects
@@
 		)
 	)
-	(label "9V_OSC_2"
+	(label "7V_OSC_1"
 		(at 411.48 312.42 0)
 		(effects
@@
 			)
 		)
-		(property "Datasheet" "https://www.digikey.ca/en/products/detail/murata-electronics/GRM21BZ71E106KE15L/13904911"
+		(property "Datasheet" "~"
 			(at 177.8 91.44 0)
 			(effects
@@
 			)
 		)
-		(property "Description" "10 µF ±10% 25V Ceramic Capacitor X7R 0805 (2012 Metric)"
+		(property "Description" "Unpolarized capacitor"
 			(at 177.8 91.44 0)
 			(effects
@@
 	(symbol
 		(lib_id "power:+5V")
+		(at 73.66 88.9 90)
+		(unit 1)
+		(exclude_from_sim no)
+		(in_bom yes)
+		(on_board yes)
+		(dnp no)
+		(fields_autoplaced yes)
+		(property "Reference" "#PWR097"
+			(at 77.47 88.9 0)
+			(effects
+				(font
+					(size 1.27 1.27)
+				)
+				(hide yes)
+			)
+		)
+		(property "Value" "+5V"
+			(at 69.85 88.8999 90)
+			(effects
+				(font
+					(size 1.27 1.27)
+				)
+				(justify left)
+			)
+		)
+		(property "Footprint" ""
+			(at 73.66 88.9 0)
+			(effects
+				(font
+					(size 1.27 1.27)
+				)
+				(hide yes)
+			)
+		)
+		(property "Datasheet" ""
+			(at 73.66 88.9 0)
+			(effects
+				(font
+					(size 1.27 1.27)
+				)
+				(hide yes)
+			)
+		)
+		(property "Description" "Power symbol creates a global label with name \"+5V\""
+			(at 73.66 88.9 0)
+			(effects
+				(font
+					(size 1.27 1.27)
+				)
+				(hide yes)
+			)
+		)
+		(pin "1"
+		)
+		(instances
+			(project "Power-Distribution-Board"
+				(path "/b6bfdd09-2ecc-401d-9031-16f8a1e99788"
+					(reference "#PWR097")
+					(unit 1)
+				)
+			)
+		)
+	)
+	(symbol
+		(lib_id "power:+5V")
 		(at 402.59 393.7 0)
 		(unit 1)
@@
 	)
 	(symbol
+		(lib_id "Power_Distribution_Board:CJS-1200TB1")
+		(at 86.36 83.82 0)
+		(unit 1)
+		(exclude_from_sim no)
+		(in_bom yes)
+		(on_board yes)
+		(dnp no)
+		(fields_autoplaced yes)
+		(property "Reference" "S3"
+			(at 93.98 78.74 0)
+			(effects
+				(font
+					(size 1.27 1.27)
+				)
+			)
+		)
+		(property "Value" "CJS-1200TB1"
+			(at 93.98 81.28 0)
+			(effects
+				(font
+					(size 1.27 1.27)
+				)
+			)
+		)
+		(property "Footprint" "Power_Distribution_Board:CJS1200TB1"
+			(at 96.266 96.774 0)
+			(effects
+				(font
+					(size 1.27 1.27)
+				)
+				(justify left top)
+				(hide yes)
+			)
+		)
+		(property "Datasheet" "https://www.digikey.ca/en/products/detail/nidec-components/CJS-1200TB1/2095031?s=N4IgTCBcDaIMICkDKBGMAGdAVAQikAugL5A"
+			(at 96.266 98.806 0)
+			(effects
+				(font
+					(size 1.27 1.27)
+				)
+				(justify left top)
+				(hide yes)
+			)
+		)
+		(property "Description" "Dip Switch SPDT Position Surface Mount Slide (Standard) Actuator 100mA"
+			(at 96.266 94.996 0)
+			(effects
+				(font
+					(size 1.27 1.27)
+				)
+				(justify left top)
+				(hide yes)
+			)
+		)
+		(pin "3"
+		)
+		(pin "1"
+		)
+		(pin "2"
+		)
+		(instances
+			(project "Power-Distribution-Board"
+				(path "/b6bfdd09-2ecc-401d-9031-16f8a1e99788"
+					(reference "S3")
+					(unit 1)
+				)
+			)
+		)
+	)
+	(symbol
 		(lib_id "Device:R")
 		(at 513.08 184.15 0)
@@
 			)
 		)
-		(property "Datasheet" "https://www.digikey.ca/en/products/detail/murata-electronics/GRM21BZ71E106KE15L/13904911"
+		(property "Datasheet" "~"
 			(at 115.57 91.44 0)
 			(effects
@@
 			)
 		)
-		(property "Description" "10 µF ±10% 25V Ceramic Capacitor X7R 0805 (2012 Metric)"
+		(property "Description" "Unpolarized capacitor"
 			(at 115.57 91.44 0)
 			(effects
@@
 			)
 		)
-		(property "Value" "13k"
+		(property "Value" "15k"
 			(at 511.81 323.8499 0)
 			(effects
@@
 			)
 		)
-		(property "Model" "ERJ-PB3B1302V"
+		(property "Model" "ERA-3AEB153V"
 			(at 509.27 322.58 0)
 			(effects
@@
 	)
 	(symbol
-		(lib_id "power:+5V")
-		(at 106.68 81.28 0)
-		(unit 1)
-		(exclude_from_sim no)
-		(in_bom yes)
-		(on_board yes)
-		(dnp no)
-		(fields_autoplaced yes)
-		(property "Reference" "#PWR021"
-			(at 106.68 85.09 0)
-			(effects
-				(font
-					(size 1.27 1.27)
-				)
-				(hide yes)
-			)
-		)
-		(property "Value" "+5V"
-			(at 106.68 76.2 0)
-			(effects
-				(font
-					(size 1.27 1.27)
-				)
-			)
-		)
-		(property "Footprint" ""
-			(at 106.68 81.28 0)
-			(effects
-				(font
-					(size 1.27 1.27)
-				)
-				(hide yes)
-			)
-		)
-		(property "Datasheet" ""
-			(at 106.68 81.28 0)
-			(effects
-				(font
-					(size 1.27 1.27)
-				)
-				(hide yes)
-			)
-		)
-		(property "Description" "Power symbol creates a global label with name \"+5V\""
-			(at 106.68 81.28 0)
-			(effects
-				(font
-					(size 1.27 1.27)
-				)
-				(hide yes)
-			)
-		)
-		(pin "1"
-		)
-		(instances
-			(project "Power-Distribution-Board"
-				(path "/b6bfdd09-2ecc-401d-9031-16f8a1e99788"
-					(reference "#PWR021")
-					(unit 1)
-				)
-			)
-		)
-	)
-	(symbol
 		(lib_id "Device:R")
 		(at 133.35 88.9 90)
@@
 			)
 		)
-		(property "Value" "182k"
+		(property "Value" "160k"
 			(at 511.81 312.4199 0)
 			(effects
@@
 			)
 		)
-		(property "Model" "ERA-3AEB1823V"
+		(property "Model" "RC0603FR-07160KL"
 			(at 509.27 311.15 0)
 			(effects
@@
 			)
 		)
-		(property "Value" "374k"
+		(property "Value" "300k"
 			(at 412.496 295.91 90)
 			(effects
@@
 			)
 		)
-		(property "Model" "RT0603BRD07374KL"
+		(property "Model" "ERA-3AEB304V"
 			(at 412.75 298.45 90)
 			(effects
@@
 			)
 		)
-		(property "Datasheet" "https://www.digikey.ca/en/products/detail/murata-electronics/GRM21BZ71E106KE15L/13904911"
+		(property "Datasheet" "~"
 			(at 304.8 69.85 0)
 			(effects
@@
 			)
 		)
-		(property "Description" "10 µF ±10% 25V Ceramic Capacitor X7R 0805 (2012 Metric)"
+		(property "Description" "Unpolarized capacitor"
 			(at 304.8 69.85 0)
 			(effects

Commit message: cleaned up schematic + readme
Other:
- note added: "IC Power Supply"
- note added: "Microcontroller (STM32)"
- note added: "Output Regulators"
- note added: "USB"
- moved on the sheet: C1, C13, C14, C15, C16, C17, C18, C19, C2, C20, C21, C22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
